File: KiCAD/ChuaCircuit/ChuaCircuit.kicad_sch (KiCad schematic)
At the start: 21 parts, among them X1 TP3, Y1 TP2

Commit message: Fixed bug with wrong GND net name
Connections:
- net at C2.1, R7.2, RV1.1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: now also OPA1.10 (+)
Changed lines of the file:
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@@
+	)
+	(junction
+		(at 95.25 66.04)
+		(diameter 0)
+		(color 0 0 0 0)
 	)
 	(junction
@@
 	(wire
 		(pts
+			(xy 90.17 66.04) (xy 95.25 66.04)
+		)
+		(stroke
+			(width 0)
+			(type default)
+		)
+	)
+	(wire
+		(pts
 			(xy 144.78 63.5) (xy 144.78 87.63)
 		)
@@
 	(wire
 		(pts
-			(xy 90.17 67.31) (xy 90.17 73.66)
-		)
-		(stroke
-			(width 0)
-			(type default)
-		)
-	)
-	(wire
-		(pts
 			(xy 161.29 76.2) (xy 157.48 76.2)
 		)
@@
 	(wire
 		(pts
+			(xy 90.17 66.04) (xy 90.17 73.66)
+		)
+		(stroke
+			(width 0)
+			(type default)
+		)
+	)
+	(wire
+		(pts
 			(xy 95.25 110.49) (xy 95.25 109.22)
 		)
@@
 		)
 		(stroke
-			(width 0)
-			(type default)
-		)
-	)
-	(wire
-		(pts
-			(xy 95.25 67.31) (xy 90.17 67.31)
-		)
-		(stroke
