File: KiCAD/ChuaCircuit/ChuaCircuit.kicad_pcb (KiCad board)
At the start: 2 copper layers, 30 x 40 mm, 21 parts, among them X1 TP3, Y1 TP2

Commit message: Fixed bug with wrong GND net name
Connections:
- C2 pad 1: Net-(C2-Pad1) -> Net-(OPA1C-+)
- OPA1 pad 10: unconnected-(OPA1C-+-Pad10) -> Net-(OPA1C-+)
- R7 pad 2: Net-(C2-Pad1) -> Net-(OPA1C-+)
- RV1 pad 1: Net-(C2-Pad1) -> Net-(OPA1C-+)
- Y1 pad 1: Net-(C2-Pad1) -> Net-(OPA1C-+)
Routing:
- net Net-(OPA1C-+): track 0.00 -> 61.5 mm
- net Net-(C2-Pad1): track 51.6 -> 0.00 mm, vias 1 -> 0
- net VCC: track 15.8 -> 0.00 mm
- net Net-(OPA1-Pad14): track 46.7 -> 54.2 mm
- net Net-(OPA1A-+): track 66.5 -> 60.2 mm
- net Net-(OPA1B--): track 19.0 -> 22.3 mm
- net GND: track 98.2 -> 96.6 mm
- net Net-(OPA1C--): track 27.9 -> 29.4 mm
- net Net-(OPA1-Pad7): track 11.4 -> 12.5 mm
- net Net-(C3-Pad1): track 18.9 -> 19.9 mm
- net Net-(OPA1-Pad1): track 25.9 -> 25.4 mm
Other:
- board text added: "Justin Nguyen's Chua Circuit 11/11/25"
