File: KiCAD/ChuaCircuit/ChuaCircuit.kicad_pcb (KiCad board)
At the start: 2 copper layers, 29.5 x 31 mm, 31 parts

Commit message: Fixed the issue with -Vcc not being connected for some reason
Parts:
- +VCC1: renamed from +VCC; value J1 -> Male_Header_1x1 2.54mm
- -VCC1: renamed from -VCC; value J1 -> Male_Header_1x1 2.54mm
- CHUA_OUT1: renamed from CHUA_OUT; value Male_Header_1x1 -> Male_Header_1x1 2.54mm
- renumbered GND to GND2, X to X1, Y to Y1, Z to Z1
Connections:
- -VCC1 pad 1: Net-(-VCC1-Pin_1) -> -VDC
- C10 pad 1: Net-(OPA2C-V-) -> -VDC
- C11 pad 1: Net-(OPA2C-V-) -> -VDC
- C6 pad 1: Net-(-VCC1-Pin_1) -> -VDC
- C7 pad 1: Net-(-VCC1-Pin_1) -> -VDC
- OPA1 pad 11: Net-(-VCC1-Pin_1) -> -VDC
- OPA2 pad 4: Net-(OPA2C-V-) -> -VDC
Routing:
- net -VDC: track 0.00 -> 28.6 mm, vias 0 -> 2
- net Net-(-VCC1-Pin_1): track 17.1 -> 0.00 mm
- net Net-(OPA2C-V-): track 12.5 -> 0.00 mm
- net Net-(OPA1A--): track 33.5 -> 21.1 mm
- net Net-(OPA1C--): track 14.7 -> 21.3 mm
- net VCC: track 48.0 -> 42.6 mm
- net Net-(OPA1C-+): track 40.7 -> 36.0 mm
- net Net-(OPA1-Pad14): track 31.5 -> 35.9 mm, vias 1 -> 2
- net Net-(OPA1D-+): track 24.9 -> 21.3 mm
- net Net-(OPA1B--): track 20.1 -> 16.5 mm
- net GND: track 83.2 -> 86.3 mm, vias 1 -> 2
- net Net-(OPA1A-+): track 74.8 -> 73.1 mm
- net Net-(C3-Pad1): track 14.7 -> 13.8 mm
